Commit message: 抓取调试一轮：链条跑通到 stage=0，物理夹持仍失败（附完整交接文档）
新增
- turtlebot3_manipulation_grasp 包（msg/srv/C++ 节点/视觉适配层/配置/launch）
- grasp_phase.py（抓取阶段唯一实现）+ dining_grasp_task.py（薄壳入口）
- HANDOFF_harness/：check_grasp_geometry.py(抓取几何自检)、vision_probe.py(视觉探针)、
  capture_grasp.py(抓取过程相机取证)、sweep_target.py(抓取点扫描)
- docs/HANDOFF_debug_state_2026-09-14.md 等交接文档

修正（每条都有现场证据，详见交接文档 §1）
- 物体碰撞箱朝向：identity → "物体 map 偏航 − 机器人 map 偏航"（原来差 90°，会把盒子顶倒）
- 抓取高度：按 URDF 真实碰撞体逐角扫描重定全部 grasp_lift；运行期加可行窗口自检
- 抓取角采样 15°→90°（原来薄盒有 14/24 个"可行但偏 15~45°"的角，手指斜着夹）
- 合爪干涉量收敛成单参数 close_hand_squeeze（当前 = 两指间距 29 mm）
- 接近方向 = 支撑面桌沿法线（原来含 AMCL 误差，实测斜 24°）；
  支撑面改为从 grasp_params.yaml 读（orchestration 与抓取侧同源）
- 最终抓取点 = 抓取点上最后一张照片（并重打时间戳）
- 视觉调用超时 60→150 s（原来超时会静默退回 1m 外的旧估计）
- 多帧投票改为"取框心中位数那一帧"；抓取模式开启 INSID3 闭集复核；
  窄词表复核也走闭集；新增"掩码法 vs 框心法"位置核对
- 删除全部 gz 真值相关代码（规则书禁止）

世界（经用户批准）
- example.world：餐桌3 的 pudding_box → tomato_soup_can（换物体对照实验）
  备份：example.world.bak_before_can

已知未解
- 夹爪能合到指令值 29 mm 而物体纹丝不动 ⇒ 合爪时两指之间没有实体；
  几何反推偏差量级 5~8 cm ⇒ 抓取点系统性偏"远"（视觉绝对位置精度问题，最优先）

File: turtlebot3_manipulation_gazebo/urdf/turtlebot3_waffle_pi.urdf.xacro (robot description, xacro)
@@ -134,4 +134,33 @@
     </inertial>
   </link>
+  <!-- ══════════ 前万向轮（本项目新增）══════════
+       为什么必须加：底盘 1.55 kg，机械臂 19.6 kg（质心还高 0.87 m），而支撑多边形
+       只有 [x=-0.177, x=0]——两个万向轮都在【后方】，驱动轮在 x=0。算下来机械臂
+       质心只要前移 0.2 mm 整车质心就越过轮轴 → 向前伸臂抓取时必然前倾（实测
+       pitch 达 0.22 rad ≈ 12.6°，导致末端偏离约 7 cm，完全抓不到物体）。
+       用位置 IK 求出能抓到桌面目标点的 57 个构型，机械臂质心 x ∈ [-0.068, +0.153]；
+       把支撑多边形前边界推到 +0.18 后允许到 +0.195，留 42 mm 余量（静态判据）。
+       这是修正模型几何，不是补偿：真实移动操作机器人前方也需要支撑点。
+       位置/几何/底面高度与既有后万向轮完全一致，保证落在同一接地平面上。 -->
+  <joint name="${prefix}caster_front_joint" type="fixed">
+    <parent link="${prefix}base_link"/>
+    <child link="${prefix}caster_front_link"/>
+    <origin xyz="0.18 0.0 -0.004" rpy="-1.57 0 0"/>
+  </joint>
+  <link name="${prefix}caster_front_link">
+    <collision>
+      <origin xyz="0 0.001 0" rpy="0 0 0"/>
+      <geometry>
+        <box size="0.030 0.009 0.020"/>
+      </geometry>
+    </collision>
+    <inertial>
+      <origin xyz="0 0 0" />
+      <mass value="0.005" />
+      <inertia ixx="0.001" ixy="0.0" ixz="0.0"
+               iyy="0.001" iyz="0.0"
+               izz="0.001" />
+    </inertial>
+  </link>
   <joint name="${prefix}imu_joint" type="fixed">
     <parent link="${prefix}base_link"/>
