Commit message: 校赛提交：抓取链修复 + 基础题计数清单可配置 + 换世界工具（10 套离线自检全绿）
一、抓取（拔高题）
  - Fortress 不支持 URDF mimic ⇒ joint2 改受控关节 + finger_mimic_relay 中继
    （此前右指物理上停在闭合端 ⇒ 两指不同步、夹持力为零）
  - 合拢轴不再依赖 AMCL 偏航：激光扫餐桌 4 条腿反解真偏航，偏差 e 注入
    grasp_node 的 object_yaw_map（C++ 侧改为每请求重读）
  - 抓取高度策略：几何自检新增【下沿余量】列（暴露 5 个类别 lift 贴住可行窗下沿）
  - 接触判据：contact/empty/unclosed + 新增 wrong_object
    （实测间距比目标窄边宽 >4 mm ⇒ 抓错物体，不算成功）
  - 视觉：调用方点类即走闭集复核；标签按实测尺寸严格纠正（三条判据）；
    「标签抖动替代」半径 0.25/0.35 → 0.10 m（0.12 m 外是另一个物体，禁止替代）
  - 观察/站位：观察位原地扫视 + 近看位沿同一法线 cmd_vel 前进（不再绕桌撞桌）；
    桌面剔除补丁（掩码吃桌面会把抓取点拉近 ~100 mm）
  - 抓取点闭环：落点核对 / 姿态核对 / 两指对称核对 / 偏置阶梯 + 跟随位移

二、基础题（导航 + 视觉识别计数）
  - 新增 config/count_items.yaml：一处配置同步三处词表
    （vision_pipeline.ITEM_NAMES/别名、insid3_review.TARGET_CLASSES、patrol_task 答案 JSON 类别）
  - 新增 scripts/count_items.py + patrol_task 接线（启动即打印生效词表，缺参考图会点名）

三、换世界 / 部署
  - launch 参数化：world:= 与 spawn_x/y/z/yaw:=（默认给文件名：
    解析顺序 原路径 → install/worlds → 源码树 worlds；找不到时打印候选并明确报错）
  - HANDOFF_harness/world_tools.py：check（体检+同步清单）/ map（由 world 直接生成
    map.pgm/yaml，不用跑 SLAM）/ status（一条命令看清当前用哪个世界与配置是否对上）
  - 附带裁判下发的两个世界：robocup_home.world 与 robocup_home_testobjects.world

四、测试与文档
  - HANDOFF_harness 离线自检 10 套（新增：扫视几何、接触重抓、桌面剔除、合拢判定、
    桌腿基准、模式判据、标签改标、构造冒烟、计数清单；另含几何自检与换世界工具）
  - docs/handoff/ 新增 4 篇（换世界 runbook / 合拢轴与抓取高度 / 计数清单 / 导航扫视与容差）

File: turtlebot3_manipulation_gazebo/ros2_control/turtlebot3_manipulation_system.ros2_control.xacro (robot description, xacro)
@@ -177,6 +177,32 @@
         </state_interface>
       </joint>
-      <!-- FR3 finger (only joint1; joint2 is URDF mimic handled by Gazebo physics) -->
+      <!-- ★ FR3 两个手指关节：**两个都必须声明成受控关节**（2026-09-18 修的真 bug）
+           背景：URDF 里 `fr3_finger_joint2` 靠 `<mimic joint="fr3_finger_joint1"/>` 联动，
+           但 **Fortress 的 sdformat12 = SDF 1.9 不支持 mimic（SDF 1.10+ 才有）**，实测：
+             $ ign sdf -p <生成的 urdf> | grep -c mimic   ⇒  **0**（整条被丢掉）
+           ⇒ joint2 在仿真里是【被动关节】：没有任何驱动（原来只声明了 joint1），
+             于是停在 URDF 默认值 0 = **闭合端**，而 joint1 的 initial_value = 0.04 = 张开 ✗
+           ⇒ 物理上"右指内侧面"永远停在夹爪中线附近（y ≈ 0），
+             而规划层（URDF 带 mimic）以为它在 y = −q
+           ⇒ 计划中的 80 mm 对称开口，物理上只有 ~40 mm 且偏离轴线 ~20 mm ✗✗
+             顶抓时右指正好落在物体【轴线上】⇒ 下降被物体顶面挡住、臂停在半路：
+               tomato_soup_can（顶 0.881 / 计划 TCP 0.868）⇒ 停在比计划高 22 mm 处
+               sugar_box     （顶 0.955 / 计划 TCP 0.9195）⇒ 高 45 mm
+             现场现象正是"指尖顶在物体顶面、伸不下去" ✓（与现场日志完全对得上）
+           修法：joint2 也声明成受控关节（位置指令 + 状态），
+                 并由 scripts/finger_mimic_relay.py 把 joint1 的值转发给它 ⇒ 两指真正对称 ✓ -->
       <joint name="fr3_finger_joint1">
+        <command_interface name="position">
+          <param name="min">0.0</param>
+          <param name="max">0.04</param>
+        </command_interface>
+        <state_interface name="position">
+          <param name="initial_value">0.04</param>
+        </state_interface>
+        <state_interface name="velocity">
+          <param name="initial_value">0.0</param>
+        </state_interface>
+      </joint>
+      <joint name="fr3_finger_joint2">
         <command_interface name="position">
           <param name="min">0.0</param>
